Commit message: save

File: example_ws/src/hector_slam/rosbot_description/rosbot_description/urdf/rosbot.xacro (robot description, xacro)
@@ -8,5 +8,5 @@
   <xacro:include filename="$(find rosbot_description)/urdf/rosbot.gazebo" />
   <xacro:include filename="$(find rosbot_description)/urdf/materials.xacro" />
-  <xacro:include filename="$(find rosbot_description)/urdf/macros.xacro" />
+  <!-- <xacro:include filename="$(find rosbot_description)/urdf/macros.xacro" /> -->
   <link name='base_link'>
     <pose>0 0 0.1 0 0 0</pose>
@@ -285,5 +285,6 @@
   <link name="camera_depth_frame">
   </link>
-  <joint name="rplidar_joint" type="fixed">
+  <!-- SickLMS100 Laser -->
+  <joint name="LMS1xx_small_joint" type="fixed">
     <axis xyz="0 1 0" />
     <origin xyz="0.02 0 0" rpy="0 0 3.14"/>
@@ -291,9 +292,28 @@
     <child link="laser"/>
   </joint>
-  <!-- rplidar Laser -->
   <link name="laser">
     <collision>
       <origin xyz="0 0 0.058" rpy="1.5707 0 4.71"/>
       <geometry>
+        <mesh filename="package://rosbot_description/meshes/LMS1xx_small.dae" scale="0.001 0.001 0.001" />
+      </geometry>
+    </collision>
+    <visual>
+      <origin xyz="0 0 0.058" rpy="1.5707 0 4.71"/>
+      <geometry>
+        <mesh filename="package://rosbot_description/meshes/LMS1xx_small.dae" scale="0.001 0.001 0.001" />
+      </geometry>
+    </visual>
+    <inertial>
+      <mass value="1e-5" />
+      <origin xyz="0 0 0.058" rpy="1.5707 0 4.71"/>
+      <inertia ixx="0" ixy="0" ixz="0" iyy="0" iyz="0" izz="0" />
+    </inertial>
+  </link>
+<!-- rplidar Laser -->
+<!--   <link name="laser">
+    <collision>
+      <origin xyz="0 0 0.058" rpy="1.5707 0 4.71"/>
+      <geometry>
         <mesh filename="package://rosbot_description/meshes/rplidar.dae" scale="0.001 0.001 0.001" />
       </geometry>
@@ -311,4 +331,10 @@
     </inertial>
   </link>
+  <joint name="rplidar_joint" type="fixed">
+    <axis xyz="0 1 0" />
+    <origin xyz="0.02 0 0" rpy="0 0 3.14"/>
+    <parent link="base_link"/>
+    <child link="laser"/>
+  </joint> -->
   <joint name="range_fl_joint" type="fixed">
     <axis xyz="0 1 0" />

Commit message: save

File: example_ws/src/hector_slam/rosbot_description/rosbot_description/urdf/rosbot.xacro (robot description, xacro)
@@ -285,6 +285,6 @@
   <link name="camera_depth_frame">
   </link>
-  <!-- SickLMS100 Laser -->
-  <joint name="LMS1xx_small_joint" type="fixed">
+  <!-- TungNV - SickLMS100 Laser -->
+<!--   <joint name="LMS1xx_small_joint" type="fixed">
     <axis xyz="0 1 0" />
     <origin xyz="0.02 0 0" rpy="0 0 3.14"/>
@@ -310,7 +310,7 @@
       <inertia ixx="0" ixy="0" ixz="0" iyy="0" iyz="0" izz="0" />
     </inertial>
-  </link>
+  </link> -->
 <!-- rplidar Laser -->
-<!--   <link name="laser">
+  <link name="laser">
     <collision>
       <origin xyz="0 0 0.058" rpy="1.5707 0 4.71"/>
@@ -336,5 +336,5 @@
     <parent link="base_link"/>
     <child link="laser"/>
-  </joint> -->
+  </joint>
   <joint name="range_fl_joint" type="fixed">
     <axis xyz="0 1 0" />
